Commit message: implemented particle filter

File: urdf/robot_model.xacro (robot description, xacro)
@@ -9,7 +9,7 @@
         <origin xyz="0.0 0.0 0.1" rpy="0.0 0 0.0"/>
         <visual name='base_visual'>
-            <origin xyz="0.0 0.0 0.2" rpy="0.0 ${pi/2} 0.0"/>
+            <origin xyz="0.0 0.0 0.2" rpy="0.0 0.0 0.0"/>
             <geometry>
-                <box size="0.2 0.6 0.6"/>
+                <box size="0.6 0.6 0.2"/>
             </geometry>
             <material name="white"/>
@@ -25,5 +25,5 @@
         </collision>
         <collision name='caster_collision'>
-            <origin xyz="0.0 -0.25 0.1" rpy="0.0 0.0 0.0"/>
+            <origin xyz="-0.25 0 0.1" rpy="0.0 0.0 0.0"/>
             <geometry>
                 <sphere radius="0.1" />
@@ -41,5 +41,5 @@
         </collision>
         <visual name='caster_visual'>
-            <origin xyz="0.0 -0.25 0.1" rpy="0.0 0.0 0.0"/>
+            <origin xyz="-0.25 0.0 0.1" rpy="0.0 0.0 0.0"/>
             <geometry>
                 <sphere radius="0.1" />
@@ -58,9 +58,9 @@
         </link>
         <joint name="lidar_joint" type="fixed">
-            <origin xyz="0 0.275 0.325" rpy="0 0 ${pi/2}"/>
+            <origin xyz="0.275 0 0.325" rpy="0 0 0"/>
             <child link="lidar_link"/>
             <parent link="base_link"/>
         </joint>
-    <xacro:wheel side="left" x="-0.325" y="0.15" z="0.1"/>
-    <xacro:wheel side="right" x="0.325" y="0.15" z="0.1"/>
+    <xacro:wheel side="left" x="0.15" y="0.325" z="0.1"/>
+    <xacro:wheel side="right" x="0.15" y="-0.325" z="0.1"/>
 </robot>

File: urdf/wheel.xacro (robot description, xacro)
@@ -21,5 +21,5 @@
     </link>
     <joint name="wheel_${side}_joint" type="continuous">
-        <origin xyz="${x} ${y} ${z}" rpy="${pi/2} 0 ${3*pi/2}"/>
+        <origin xyz="${x} ${y} ${z}" rpy="${-pi/2} 0 0"/>
         <child link="wheel_${side}"/>
         <axis xyz="0 0 1"/>
